File: interphase.kicad_pcb (KiCad board)
At the start: 2 copper layers, 134.6 x 105.4 mm, 107 parts, among them SW1 MOM-SPST, SW10 MOM-SPST, SW11 MOM-SPST, SW12 MOM-SPST, SW13 MOM-SPST, SW14 MOM-SPST, SW15 MOM-SPST, SW16 MOM-SPST, SW17 MOM-SPST, SW18 MOM-SPST, SW19 MOM-SPST, SW2 MOM-SPST, SW20 MOM-SPST, SW21 MOM-SPST, SW22 MOM-SPST, SW23 MOM-SPST, SW24 MOM-SPST, SW25 MOM-SPST, SW26 MOM-SPST, SW27 MOM-SPST, SW28 MOM-SPST, SW29 MOM-SPST, SW3 MOM-SPST, SW30 MOM-SPST, SW31 MOM-SPST, SW32 MOM-SPST, SW33 MOM-SPST, SW34 MOM-SPST, SW35 MOM-SPST, SW36 MOM-SPST, SW4 MOM-SPST, SW5 MOM-SPST, SW6 MOM-SPST, SW7 MOM-SPST, SW8 MOM-SPST, SW9 MOM-SPST, U2 MCP1640

Commit message: some work
Parts:
- removed REF** (x33): CHERRY-MX, Misc:CHERRY-MX
- moved SW2 185.3 mm to (81.3, 47.0)
- moved SW3 161.6 mm to (81.3, 66.0)
- moved SW32 127.4 mm to (195.6, 44.5)
- moved SW1 126.0 mm to (77.5, 146.1)
- moved SW27 125.0 mm to (176.5, 36.8)
- moved D31 123.9 mm to (201.9, 53.3), turned to 180 degrees
- moved SW22 121.0 mm to (157.5, 34.3)
- moved D26 119.8 mm to (182.9, 45.7), turned to 180 degrees
- moved SW17 114.9 mm to (138.4, 36.8)
- moved D21 114.4 mm to (163.8, 43.2), turned to 180 degrees
- moved SW33 112.0 mm to (195.6, 63.5)
- moved D32 109.5 mm to (201.9, 72.4), turned to 180 degrees
- moved SW28 107.9 mm to (176.5, 55.9)
- moved SW7 107.1 mm to (100.3, 47.0)
- moved D16 107.0 mm to (144.8, 45.7), turned to 180 degrees
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Other:
- board size 134.6 x 105.4 mm -> 250.2 x 189.2 mm

Commit message: routing
Parts:
- removed D35, D9: D, Diodes_SMD:D_MiniMELF
- removed SW1, SW10, SW36: MOM-SPST, Misc:CHERRY-MX
- added BT1: Battery_Cell, Misc:KEYSTONE-82_AAA_battery-clip, F.Cu at (100.3, 29.2)
- added C1: 4,7µF, Capacitors_SMD:C_0805_HandSoldering, B.Cu at (334.0, 20.4)
- added C2: 10µF, Capacitors_SMD:C_0805_HandSoldering, B.Cu at (334.0, 17.8)
- added D1: D, Diodes_SMD:D_MiniMELF, B.Cu at (90.2, 50.8)
- added D10: D, Diodes_SMD:D_MiniMELF, B.Cu at (110.5, 127.0)
- added D11: D, Diodes_SMD:D_MiniMELF, B.Cu at (128.3, 45.7)
- added D12: D, Diodes_SMD:D_MiniMELF, B.Cu at (129.5, 65.2)
- added D13: D, Diodes_SMD:D_MiniMELF, B.Cu at (129.5, 83.8)
- added D14: D, Diodes_SMD:D_MiniMELF, B.Cu at (129.5, 102.9)
- added D15: D, Diodes_SMD:D_MiniMELF, B.Cu at (129.5, 126.5)
- added D16: D, Diodes_SMD:D_MiniMELF, B.Cu at (147.3, 40.6)
- added D17: D, Diodes_SMD:D_MiniMELF, B.Cu at (148.6, 60.2)
- added D18: D, Diodes_SMD:D_MiniMELF, B.Cu at (148.6, 79.2)
- added D19: D, Diodes_SMD:D_MiniMELF, B.Cu at (148.6, 97.8)
- added D2: D, Diodes_SMD:D_MiniMELF, B.Cu at (90.2, 69.8)
- added D20: D, Diodes_SMD:D_MiniMELF, B.Cu at (148.6, 126.5)
- added D21: D, Diodes_SMD:D_MiniMELF, B.Cu at (166.4, 39.4)
- added D22: D, Diodes_SMD:D_MiniMELF, B.Cu at (167.6, 58.9)
- added D23: D, Diodes_SMD:D_MiniMELF, B.Cu at (167.6, 77.5)
- added D24: D, Diodes_SMD:D_MiniMELF, B.Cu at (167.6, 96.5)
- added D25: D, Diodes_SMD:D_MiniMELF, B.Cu at (176.5, 133.3)
- added D26: D, Diodes_SMD:D_MiniMELF, B.Cu at (185.9, 47.0)
- added D27: D, Diodes_SMD:D_MiniMELF, B.Cu at (185.4, 66.5)
- added D28: D, Diodes_SMD:D_MiniMELF, B.Cu at (185.4, 85.6)
- added D29: D, Diodes_SMD:D_MiniMELF, B.Cu at (185.4, 102.9)
- added D3: D, Diodes_SMD:D_MiniMELF, B.Cu at (91.4, 89.4)
- added D30: D, Diodes_SMD:D_MiniMELF, B.Cu at (203.7, 132.1)
- added D31: D, Diodes_SMD:D_MiniMELF, B.Cu at (204.5, 48.3)
- added D32: D, Diodes_SMD:D_MiniMELF, B.Cu at (208.3, 67.8)
- added D33: D, Diodes_SMD:D_MiniMELF, B.Cu at (208.3, 86.8)
- added D34: D, Diodes_SMD:D_MiniMELF, B.Cu at (207.0, 105.4)
- added D36: LED, LEDs:LED_1206, B.Cu at (278.1, 11.5)
- added D36: LED, LEDs:LED_1206, F.Cu at (125.7, 29.6)
- added D4: D, Diodes_SMD:D_MiniMELF, B.Cu at (102.9, 104.1)
- added D5: D, Diodes_SMD:D_MiniMELF, B.Cu at (91.4, 126.5)
- added D6: D, Diodes_SMD:D_MiniMELF, B.Cu at (109.2, 50.8)
- added D7: D, Diodes_SMD:D_MiniMELF, B.Cu at (110.5, 70.3)
- added D8: D, Diodes_SMD:D_MiniMELF, B.Cu at (110.5, 88.9)
- added J1: Conn_01x04_Male, Pin_Headers:Pin_Header_Angled_1x04_Pitch2.54mm, B.Cu at (259.1, 15.3)
- added J1: Conn_01x04_Male, Pin_Headers:Pin_Header_Angled_1x04_Pitch2.54mm, F.Cu at (232.4, 34.3)
- added L1: 4,7µH, SMD_Packages:SMD-1206_Pol, B.Cu at (278.5, 7.67)
- added L1: 4,7µH, SMD_Packages:SMD-1206_Pol, F.Cu at (323.0, 14.0)
- added R1: 536K, Resistors_SMD:R_0805, B.Cu at (273.1, 14.0)
- added R1: 536K, Resistors_SMD:R_0805, F.Cu at (317.5, 7.62)
- added R2: 309K, Resistors_SMD:R_0805, B.Cu at (273.1, 8.94)
- added R2: 309K, Resistors_SMD:R_0805, F.Cu at (317.5, 12.7)
- added R3: 100K, Resistors_SMD:R_0805, B.Cu at (273.1, 3.86)
- added R3: 100K, Resistors_SMD:R_0805, F.Cu at (317.5, 17.8)
- added R4: R, Resistors_SMD:R_0805, B.Cu at (273.1, -1.22)
- added R4: R, Resistors_SMD:R_0805, F.Cu at (317.5, 22.9)
- added U1: Core51822B, Misc:Core51822(B), B.Cu at (193.0, 119.4)
- added U1: Core51822B, Misc:Core51822(B), F.Cu at (193.0, 119.4)
- added U2: MCP1640, TO_SOT_Packages_SMD:SOT-23-6, B.Cu at (334.0, 14.0)
- SW11, SW12, SW13, SW14, SW15, SW16, SW17, SW18, SW19, SW2, SW20, SW21, SW22, SW23, SW24, SW25, SW26, SW27, SW28, SW29, SW3, SW30, SW31, SW32, SW33, SW34, SW35, SW4, SW6, SW7, SW8, SW9: footprint Misc:CHERRY-MX -> Misc:CHERRY-MX_double_bo
- SW5: footprint Misc:CHERRY-MX -> Misc:CHERRY-MX_double_bo_2u
- moved U2 52.1 mm to (155.1, 110.8)
- moved SW31 24.9 mm to (195.1, 139.7), turned to 330 degrees
- moved D30 19.1 mm to (201.9, 132.1), turned to 0 degrees
- moved D4 16.6 mm to (101.6, 104.1), turned to 90 degrees
- moved D25 11.5 mm to (175.3, 130.8)
- moved SW5 9.53 mm to (90.8, 104.1)
- moved SW26 8.89 mm to (165.3, 127.5), turned to 345 degrees
- moved D11 8.03 mm to (128.3, 45.7), turned to 90 degrees
- moved D12 8.03 mm to (128.3, 64.8), turned to 90 degrees
- moved D13 8.03 mm to (128.3, 83.8), turned to 90 degrees
- moved D14 8.03 mm to (128.3, 102.9), turned to 90 degrees
- moved D15 5.68 mm to (128.3, 127.0), turned to 90 degrees
- moved D2 5.68 mm to (90.2, 69.8), turned to 90 degrees
- moved D5 5.68 mm to (90.2, 127.0), turned to 90 degrees
- moved D1 5.68 mm to (90.2, 50.8), turned to 90 degrees
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Connections:
- D12 pad 1: Net-(D12-Pad1) -> Net-(D11-Pad1)
- D13 pad 1: Net-(D13-Pad1) -> Net-(D11-Pad1)
- D14 pad 1: Net-(D14-Pad1) -> Net-(D11-Pad1)
- D15 pad 1: Net-(D15-Pad1) -> Net-(D11-Pad1)
- D18 pad 1: Net-(D18-Pad1) -> Net-(D16-Pad1)
- D19 pad 1: Net-(D19-Pad1) -> Net-(D16-Pad1)
- D20 pad 1: Net-(D20-Pad1) -> Net-(D16-Pad1)
- D22 pad 1: Net-(D22-Pad1) -> Net-(D21-Pad1)
- D23 pad 1: Net-(D23-Pad1) -> Net-(D21-Pad1)
- D24 pad 1: Net-(D24-Pad1) -> Net-(D21-Pad1)
- D25 pad 1: Net-(D25-Pad1) -> Net-(D21-Pad1)
- D27 pad 1: Net-(D27-Pad1) -> Net-(D26-Pad1)
- D28 pad 1: Net-(D28-Pad1) -> Net-(D26-Pad1)
- D29 pad 1: Net-(D29-Pad1) -> Net-(D26-Pad1)
- D30 pad 1: Net-(D30-Pad1) -> Net-(D26-Pad1)
- D32 pad 1: Net-(D32-Pad1) -> Net-(D31-Pad1)
- D33 pad 1: Net-(D33-Pad1) -> Net-(D31-Pad1)
- D34 pad 1: Net-(D34-Pad1) -> Net-(D31-Pad1)
- D6 pad 1: Net-(D6-Pad1) -> Net-(D10-Pad1)
- D7 pad 1: Net-(D7-Pad1) -> Net-(D10-Pad1)
- D8 pad 1: Net-(D8-Pad1) -> Net-(D10-Pad1)
- U2 pad 3: Net-(R3-Pad1) -> Net-(BT1-Pad1)
Routing:
- net Net-(SW13-Pad1): track 0.00 -> 237.5 mm
- net Net-(SW14-Pad1): track 0.00 -> 237.5 mm
- net Net-(SW12-Pad1): track 0.00 -> 237.5 mm
- net Net-(SW15-Pad1): track 0.00 -> 233.3 mm
- net Net-(SW11-Pad1): track 0.00 -> 226.8 mm
- net Net-(D1-Pad1): track 0.00 -> 128.1 mm, vias 0 -> 5
- net Net-(D21-Pad1): track 0.00 -> 113.4 mm, vias 0 -> 5
- net Net-(D31-Pad1): track 0.00 -> 102.7 mm, vias 0 -> 4
- net Net-(D11-Pad1): track 0.00 -> 93.6 mm, vias 0 -> 5
- net Net-(D26-Pad1): track 0.00 -> 91.7 mm, vias 0 -> 4
- net Net-(D10-Pad1): track 0.00 -> 86.5 mm, vias 0 -> 4
- net Net-(D16-Pad1): track 0.00 -> 58.6 mm, vias 0 -> 4
- net Net-(D30-Pad2): track 0.00 -> 22.0 mm
- net Net-(D21-Pad2): track 0.00 -> 20.5 mm
- net Net-(D31-Pad2): track 0.00 -> 18.1 mm
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Other:
- board size 250.2 x 189.2 mm -> 32.3 x 14.8 mm

Commit message: wololo
Parts:
- SW11, SW12, SW13, SW14, SW15, SW16, SW17, SW18, SW19, SW2, SW20, SW21, SW22, SW23, SW24, SW25, SW26, SW27, SW28, SW29, SW3, SW30, SW31, SW32, SW33, SW34, SW35, SW4, SW6, SW7, SW8, SW9: footprint Misc:CHERRY-MX_double_bo -> Misc:CHERRY-MX_double_bo_nodiode
- SW5: footprint Misc:CHERRY-MX_double_bo_2u -> Misc:CHERRY-MX_double_bo_2u_nodiode
- moved C1 188.2 mm to (268.0, 27.9)
- moved C2 188.2 mm to (268.0, 30.5)
- moved U2 153.1 mm to (287.2, 33.3)
- moved U1 115.4 mm to (306.1, 142.9)
- moved U1 80.9 mm to (273.7, 112.4)
- moved D32 3.84 mm to (204.5, 67.3)
- moved D33 3.84 mm to (204.5, 86.4)
- moved D25 2.84 mm to (175.3, 130.8)
- moved D34 2.54 mm to (204.5, 105.4)
- moved D30 1.75 mm to (201.9, 132.1)
- moved D17 1.36 mm to (147.3, 59.7)
- moved D18 1.36 mm to (147.3, 78.7)
- moved D20 1.36 mm to (147.3, 127.0)
- moved D5 1.36 mm to (90.2, 127.0)
- moved D7 1.36 mm to (109.2, 69.8)
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Connections:
- D17 pad 1: Net-(D17-Pad1) -> Net-(D16-Pad1) (x2)
Routing:
- net Net-(SW13-Pad1): track 237.5 -> 0.00 mm
- net Net-(SW14-Pad1): track 237.5 -> 0.00 mm
- net Net-(SW12-Pad1): track 237.5 -> 0.00 mm
- net Net-(SW15-Pad1): track 233.3 -> 0.00 mm
- net Net-(SW11-Pad1): track 226.8 -> 0.00 mm
- net Net-(D1-Pad1): track 128.1 -> 0.00 mm, vias 5 -> 0
- net Net-(D21-Pad1): track 113.4 -> 0.00 mm, vias 5 -> 0
- net Net-(D31-Pad1): track 102.7 -> 0.00 mm, vias 4 -> 0
- net Net-(D11-Pad1): track 93.6 -> 0.00 mm, vias 5 -> 0
- net Net-(D26-Pad1): track 91.7 -> 0.00 mm, vias 4 -> 0
- net Net-(D10-Pad1): track 86.5 -> 0.00 mm, vias 4 -> 0
- net Net-(D16-Pad1): track 58.6 -> 0.00 mm, vias 4 -> 0
- net Net-(D30-Pad2): track 22.0 -> 0.00 mm
- net Net-(D21-Pad2): track 20.5 -> 0.00 mm
- net Net-(D31-Pad2): track 18.1 -> 0.00 mm
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Other:
- board size 32.3 x 14.8 mm -> 94 x 111.8 mm

Commit message: repositioning and routing
Parts:
- moved U1 250.3 mm to (85.1, 25.4), turned to 270 degrees
- moved U1 207.7 mm to (85.1, 25.4), turned to 90 degrees
- moved D36 98.5 mm to (218.4, -3.81)
- moved BT1 26.9 mm to (125.7, 20.3)
- moved D26 6.35 mm to (185.4, 40.6), turned to 90 degrees (x2)
- moved D27 6.35 mm to (185.4, 59.7), turned to 90 degrees
- moved D28 6.35 mm to (185.4, 78.7), turned to 90 degrees (x2)
- moved D29 6.35 mm to (185.4, 97.8), turned to 90 degrees (x2)
- moved D27 6.32 mm to (185.4, 59.7), turned to 90 degrees
- moved D12 2.54 mm to (128.3, 67.3) (x2)
- moved D13 2.54 mm to (128.3, 86.4)
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Routing:
- net Net-(D1-Pad1): track 0.00 -> 58.2 mm
Other:
- board size 94 x 111.8 mm -> 32.3 x 14.8 mm

Commit message: routing
Parts:
- removed the C1 at (334.0, 20.4)
- removed the C2 at (334.0, 17.8)
- removed D36 (x2): LED, LEDs:LED_1206
- removed the J1 at (259.1, 15.3)
- removed the L1 at (278.5, 7.67)
- removed the R1 at (273.1, 14.0)
- removed the R2 at (273.1, 8.94)
- removed R3 (x2): 100K, Resistors_SMD:R_0805
- removed R4 (x2): R, Resistors_SMD:R_0805
- removed the U1 at (85.1, 25.4)
- removed the U2 at (334.0, 14.0)
- added C3: 4,7µF, Capacitors_SMD:C_0805_HandSoldering, B.Cu at (123.2, 30.5)
- added C4: 10µF, Capacitors_SMD:C_0805_HandSoldering, B.Cu at (108.0, 36.8)
- added L2: 4,7µH, SMD_Packages:SMD-1206_Pol, B.Cu at (119.4, 30.5)
- added R6: 536K, Resistors_SMD:R_0805, B.Cu at (109.2, 33.0)
- added R7: 309K, Resistors_SMD:R_0805, B.Cu at (113.0, 34.3)
- added U3: MCP1640, TO_SOT_Packages_SMD:SOT-23-6, B.Cu at (113.2, 32.1)
- added U4: Core51822B, Misc:Core51822(B), B.Cu at (84.5, 24.1)
- moved R2 205.6 mm to (113.0, 34.3), turned to 180 degrees
- moved R1 202.2 mm to (116.8, 32.7), turned to 270 degrees
- moved L1 201.8 mm to (121.9, 31.8), turned to 90 degrees
- moved U2 174.2 mm to (113.0, 31.8)
- moved C1 161.4 mm to (106.7, 33.0), turned to 90 degrees
- moved C2 158.8 mm to (109.2, 30.5), turned to 270 degrees
- moved J1 152.4 mm to (80.6, 20.3), turned to 90 degrees
- moved D30 32.5 mm to (185.4, 104.1), turned to 270 degrees (x2)
- moved D25 30.5 mm to (166.4, 101.6), turned to 270 degrees (x2)
- moved U1 1.42 mm to (84.5, 24.1), turned to 0 degrees
Connections:
- net Net-(BT1-Pad1) renamed +BATT
- U1 pad 10: Net-(U1-Pad10) -> Net-(SW12-Pad1)
- U1 pad 23: Net-(D31-Pad1) -> Net-(U1-Pad23)
- U1 pad 24: Net-(D26-Pad1) -> Net-(U1-Pad24)
- U1 pad 25: Net-(D21-Pad1) -> Net-(D1-Pad1)
- U1 pad 26: Net-(D16-Pad1) -> Net-(D10-Pad1)
- U1 pad 28: Net-(D10-Pad1) -> Net-(D16-Pad1)
- U1 pad 29: Net-(D1-Pad1) -> Net-(D21-Pad1)
- U1 pad 30: Net-(SW11-Pad1) -> Net-(D26-Pad1)
- U1 pad 31: Net-(J1-Pad2) -> Net-(J1-Pad3)
- U1 pad 32: Net-(J1-Pad3) -> Net-(J1-Pad2)
- U1 pad 33: Net-(SW15-Pad1) -> Net-(D31-Pad1)
- U1 pad 34: Net-(SW14-Pad1) -> Net-(U1-Pad34)
- U1 pad 35: Net-(SW13-Pad1) -> Net-(U1-Pad35)
- U1 pad 36: Net-(SW12-Pad1) -> Net-(U1-Pad36)
- U1 pad 4: Net-(U1-Pad4) -> Net-(SW11-Pad1)
- U1 pad 5: Net-(U1-Pad5) -> Net-(SW15-Pad1)
- U1 pad 6: Net-(U1-Pad6) -> Net-(SW14-Pad1)
- U1 pad 9: Net-(U1-Pad9) -> Net-(SW13-Pad1)
Routing:
- net Net-(SW11-Pad1): track 0.00 -> 320.8 mm, vias 0 -> 1
- net Net-(SW15-Pad1): track 0.00 -> 311.8 mm, vias 0 -> 1
- net Net-(SW14-Pad1): track 0.00 -> 294.1 mm, vias 0 -> 1
- net Net-(SW13-Pad1): track 0.00 -> 277.6 mm, vias 0 -> 1
- net Net-(SW12-Pad1): track 0.00 -> 250.5 mm, vias 0 -> 1
- net Net-(D31-Pad1): track 0.00 -> 214.7 mm, vias 0 -> 5
- net Net-(D26-Pad1): track 0.00 -> 197.2 mm, vias 0 -> 5
- net Net-(D16-Pad1): track 0.00 -> 184.9 mm, vias 0 -> 6
- net Net-(D21-Pad1): track 0.00 -> 176.2 mm, vias 0 -> 5
- net Net-(D11-Pad1): track 0.00 -> 167.7 mm, vias 0 -> 6
- net Net-(D10-Pad1): track 0.00 -> 140.0 mm, vias 0 -> 5
- net GND: track 0.00 -> 124.1 mm, vias 0 -> 1
- net +3V3: track 0.00 -> 109.0 mm, vias 0 -> 1
- net Net-(D1-Pad1): track 58.2 -> 161.8 mm, vias 0 -> 6
- net +BATT: track 0.00 -> 99.3 mm, vias 0 -> 7
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
Commit message: more routing
Routing:
- net GND: track 124.1 -> 146.4 mm, vias 1 -> 2
- net Net-(SW13-Pad1): track 277.6 -> 270.4 mm
- net Net-(D5-Pad2): track 13.7 -> 11.1 mm, vias 1 -> 0
- net Net-(SW12-Pad1): track 250.5 -> 248.2 mm
- net +BATT: track 99.3 -> 100.3 mm, vias 7 -> 8
- net Net-(D31-Pad1): track 214.7 -> 214.0 mm
- net Net-(SW14-Pad1): track 294.1 -> 293.4 mm
- net Net-(D4-Pad2): track 13.2 -> 12.6 mm
Other:
- board size 32.3 x 14.8 mm -> 139.7 x 141 mm
- net class nrf added: clearance 0.1, trace_width 0.25, via_dia 0.6, via_drill 0.4

Commit message: re-routing
Parts:
- SW26, SW31: footprint Misc:CHERRY-MX_double_bo_nodiode -> Misc:CHERRY-MX_double_bo_1_5u
- moved J1 162.8 mm to (205.7, 124.5), turned to 0 degrees
- moved U1 146.4 mm to (195.6, 119.4), turned to 270 degrees
- moved U4 146.4 mm to (195.6, 119.4), turned to 90 degrees
- moved C2 92.9 mm to (160.5, 108.0), turned to 90 degrees
- moved L2 88.9 mm to (161.5, 108.7), turned to 90 degrees
- moved R7 88.4 mm to (158.2, 110.2), turned to 90 degrees
- moved R6 88.1 mm to (151.6, 110.2)
- moved U2 88.1 mm to (154.9, 109.2)
- moved R1 87.9 mm to (158.2, 110.2)
- moved U3 87.7 mm to (154.9, 109.2)
- moved C1 87.2 mm to (154.9, 105.7), turned to 180 degrees
- moved R2 85.2 mm to (151.6, 110.2), turned to 90 degrees
- moved C4 82.3 mm to (149.4, 108.0), turned to 90 degrees
- moved C3 81.6 mm to (154.9, 105.7), turned to 0 degrees
- moved L1 81.3 mm to (148.1, 108.7)
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Routing:
- net Net-(SW11-Pad1): track 320.8 -> 151.9 mm, vias 1 -> 0
- net Net-(D31-Pad1): track 214.0 -> 72.3 mm, vias 5 -> 4
- net Net-(D26-Pad1): track 197.2 -> 79.1 mm, vias 5 -> 4
- net Net-(D16-Pad1): track 184.9 -> 81.1 mm, vias 6 -> 5
- net +3V3: track 109.0 -> 9.22 mm, vias 1 -> 0
- net Net-(D21-Pad1): track 176.2 -> 79.4 mm, vias 5 -> 4
- net Net-(SW15-Pad1): track 311.6 -> 228.5 mm, vias 1 -> 0
- net Net-(D11-Pad1): track 167.7 -> 100.8 mm, vias 6 -> 5
- net Net-(SW14-Pad1): track 293.4 -> 231.4 mm, vias 1 -> 0
- net Net-(D10-Pad1): track 140.0 -> 92.1 mm, vias 5 -> 4
- net Net-(D30-Pad2): track 58.8 -> 12.2 mm
- net +BATT: track 100.3 -> 146.2 mm, vias 8 -> 2
- net Net-(SW13-Pad1): track 270.4 -> 231.4 mm, vias 1 -> 0
- net Net-(D1-Pad1): track 161.8 -> 131.3 mm, vias 6 -> 5
- net Net-(D25-Pad2): track 40.8 -> 12.0 mm
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Other:
- board size 139.7 x 141 mm -> 49.5 x 10.8 mm
- net class Bat added: clearance 0.2, trace_width 0.4, via_dia 0.6, via_drill 0.4
- net class nrf removed

Commit message: finish routing
Parts:
- moved J1 9.16 mm to (200.7, 116.8)
Connections:
- U1 pad 10: Net-(SW12-Pad1) -> Net-(SW11-Pad1)
- U1 pad 13: Net-(U1-Pad13) -> Net-(D31-Pad1)
- U1 pad 14: Net-(U1-Pad14) -> Net-(D26-Pad1)
- U1 pad 16: Net-(U1-Pad16) -> Net-(D21-Pad1)
- U1 pad 17: Net-(U1-Pad17) -> Net-(D16-Pad1)
- U1 pad 18: Net-(U1-Pad18) -> Net-(D11-Pad1)
- U1 pad 19: Net-(U1-Pad19) -> Net-(D10-Pad1)
- U1 pad 2: Net-(U1-Pad2) -> Net-(SW15-Pad1)
- U1 pad 20: Net-(U1-Pad20) -> Net-(D1-Pad1)
- U1 pad 25: Net-(D1-Pad1) -> Net-(U1-Pad25)
- U1 pad 26: Net-(D10-Pad1) -> Net-(U1-Pad26)
- U1 pad 27: Net-(D11-Pad1) -> Net-(U1-Pad27)
- U1 pad 28: Net-(D16-Pad1) -> Net-(U1-Pad28)
- U1 pad 29: Net-(D21-Pad1) -> Net-(U1-Pad29)
- U1 pad 3: Net-(U1-Pad3) -> Net-(SW14-Pad1)
- U1 pad 30: Net-(D26-Pad1) -> Net-(U1-Pad30)
- U1 pad 33: Net-(D31-Pad1) -> Net-(U1-Pad33)
- U1 pad 4: Net-(SW11-Pad1) -> Net-(SW13-Pad1)
- U1 pad 5: Net-(SW15-Pad1) -> Net-(U1-Pad5)
- U1 pad 6: Net-(SW14-Pad1) -> Net-(U1-Pad6)
- U1 pad 9: Net-(SW13-Pad1) -> Net-(SW12-Pad1)
- U4 pad 10: Net-(D1-Pad1) -> Net-(U4-Pad10)
- U4 pad 17: Net-(U4-Pad17) -> Net-(D1-Pad1)
- U4 pad 18: Net-(U4-Pad18) -> Net-(D10-Pad1)
- U4 pad 19: Net-(U4-Pad19) -> Net-(D11-Pad1)
- U4 pad 2: Net-(D31-Pad1) -> Net-(U4-Pad2)
- U4 pad 20: Net-(U4-Pad20) -> Net-(D16-Pad1)
- U4 pad 21: Net-(U4-Pad21) -> Net-(D21-Pad1)
- U4 pad 23: Net-(U4-Pad23) -> Net-(D26-Pad1)
- U4 pad 24: Net-(U4-Pad24) -> Net-(D31-Pad1)
- U4 pad 25: Net-(SW12-Pad1) -> Net-(U4-Pad25)
- U4 pad 26: Net-(SW13-Pad1) -> Net-(U4-Pad26)
- U4 pad 27: Net-(SW14-Pad1) -> Net-(SW11-Pad1)
- U4 pad 28: Net-(SW15-Pad1) -> Net-(SW12-Pad1)
- U4 pad 29: Net-(SW11-Pad1) -> Net-(U4-Pad29)
- U4 pad 3: Net-(D26-Pad1) -> Net-(U4-Pad3)
- U4 pad 33: Net-(U4-Pad33) -> Net-(SW13-Pad1)
- U4 pad 34: Net-(U4-Pad34) -> Net-(SW14-Pad1)
- U4 pad 35: Net-(U4-Pad35) -> Net-(SW15-Pad1)
- U4 pad 4: Net-(D21-Pad1) -> Net-(U4-Pad4)
- U4 pad 5: Net-(D16-Pad1) -> Net-(U4-Pad5)
- U4 pad 6: Net-(D11-Pad1) -> Net-(U4-Pad6)
- U4 pad 9: Net-(D10-Pad1) -> Net-(U4-Pad9)
Routing:
- net Net-(SW12-Pad1): track 231.7 -> 355.2 mm, vias 0 -> 1
- net GND: track 120.0 -> 237.8 mm, vias 0 -> 7
- net Net-(SW11-Pad1): track 151.9 -> 253.0 mm, vias 0 -> 3
- net Net-(SW13-Pad1): track 231.4 -> 327.8 mm, vias 0 -> 1
- net +BATT: track 146.2 -> 237.8 mm, vias 2 -> 9
- net Net-(D1-Pad1): track 131.3 -> 213.8 mm, vias 5 -> 7
- net +3V3: track 9.22 -> 90.0 mm, vias 0 -> 4
- net Net-(D10-Pad1): track 92.1 -> 171.4 mm, vias 4 -> 6
- net Net-(SW14-Pad1): track 231.4 -> 306.4 mm, vias 0 -> 1
- net Net-(D16-Pad1): track 81.1 -> 156.0 mm, vias 5 -> 7
- net Net-(D11-Pad1): track 100.8 -> 161.4 mm, vias 5 -> 7
- net Net-(D30-Pad2): track 12.2 -> 64.6 mm, vias 1 -> 2
- net Net-(SW15-Pad1): track 228.5 -> 279.6 mm, vias 0 -> 1
- net Net-(D31-Pad1): track 72.3 -> 109.3 mm, vias 4 -> 5
- net Net-(D21-Pad1): track 79.4 -> 113.3 mm, vias 4 -> 5
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