File: interphase.sch (KiCad schematic (older format))
At the start: 1 part

Commit message: schematic preversion and layout preversion
Parts:
- added BT1: Battery_Cell, symbol Battery_Cell
- added C1: 4,7µF, Capacitors_SMD:C_0805_HandSoldering, symbol C
- added C2: 10µF, Capacitors_SMD:C_0805_HandSoldering, symbol C
- added D1, D10, D11, D12, D13, D14, D15, D16, D17, D18, D19, D2, D20, D21, D22, D23, D24, D25, D26, D27, D28, D29, D3, D30, D31, D32, D33, D34, D35, D4, D5, D6, D7, D8, D9: D, Diodes_SMD:D_MiniMELF, symbol D
- added L1: 4,7µH, symbol L
- added R1: 536K, symbol R
- added R2: 309K, symbol R
- added R3: 100K, symbol R
- added SW1, SW10, SW11, SW12, SW13, SW14, SW15, SW16, SW17, SW18, SW19, SW2, SW20, SW21, SW22, SW23, SW24, SW25, SW26, SW27, SW28, SW29, SW3, SW30, SW31, SW32, SW33, SW34, SW35, SW36, SW4, SW5, SW6, SW7, SW8, SW9: MOM-SPST, Misc:CHERRY-MX, symbol MOM-SPST
- added U2: MCP1640, TO_SOT_Packages_SMD:SOT-23-6, symbol MCP1640
- gave numbers to parts that had none: 1
Connections:
- net GND: now reaches U1.1 (GND)
- net GND: now also U1.11 (GND), BT1.2 (-), C1.2, C2.2, R2.2, R3.2, U2.2 (GND)
- net +3V3: now reaches U1.12 (VCC)
- net +3V3: now also C2.1, R1.1, U2.5 (VOUT)
- net at U1.15 (P01): now also BT1.1 (+), C1.1, L1.1, SW1.1, U2.6 (VIN)
- net at U1.23 (P09): now also D31.1 (K)
- net at U1.24 (P10): now also D26.1 (K)
- net at U1.25 (P11): now also D21.1 (K)
- net at U1.26 (P12): now also D16.1 (K)
- net at U1.27 (P13): now also D11.1 (K)
- net at U1.28 (P14): now also D6.1 (K)
- net at U1.29 (P15): now also D1.1 (K), D2.1 (K), D3.1 (K), D4.1 (K), D5.1 (K)
- net at U1.30 (P16): now also SW11.1, SW16.1, SW21.1, SW26.1, SW31.1, SW36.1, SW6.1
- net at U1.33 (P17): now also SW10.1, SW15.1, SW20.1, SW25.1, SW30.1, SW35.1, SW5.1
- net at U1.34 (P18): now also SW14.1, SW19.1, SW24.1, SW29.1, SW34.1, SW4.1, SW9.1
- net at U1.35 (P19): now also SW13.1, SW18.1, SW23.1, SW28.1, SW3.1, SW33.1, SW8.1
- net at U1.36 (P20): now also SW12.1, SW17.1, SW2.1, SW22.1, SW27.1, SW32.1, SW7.1
- new net: L1.2, U2.1 (SW)
- new net: R3.1, SW1.2, U2.3 (EN)
- new net: R1.2, R2.1, U2.4 (VFB)
- new net: D31.2 (A), SW32.2
- new net: D26.2 (A), SW27.2
- new net: D21.2 (A), SW22.2
- new net: D16.2 (A), SW17.2
- new net: D11.2 (A), SW12.2
- new net: D6.2 (A), SW7.2
- new net: D1.2 (A), SW2.2
- new net: D32.2 (A), SW33.2
- new net: D27.2 (A), SW28.2
- new net: D22.2 (A), SW23.2
- new net: D17.2 (A), SW18.2
- new net: D12.2 (A), SW13.2
- new net: D7.2 (A), SW8.2
- new net: D2.2 (A), SW3.2
- new net: D33.2 (A), SW34.2
- new net: D28.2 (A), SW29.2
- new net: D23.2 (A), SW24.2
- new net: D18.2 (A), SW19.2
- new net: D13.2 (A), SW14.2
- new net: D8.2 (A), SW9.2
- new net: D3.2 (A), SW4.2
- new net: D34.2 (A), SW35.2
- new net: D29.2 (A), SW30.2
- new net: D24.2 (A), SW25.2
- new net: D19.2 (A), SW20.2
- new net: D14.2 (A), SW15.2
- new net: D9.2 (A), SW10.2
- new net: D4.2 (A), SW5.2
- new net: D35.2 (A), SW36.2
- new net: D30.2 (A), SW31.2
- new net: D25.2 (A), SW26.2
- new net: D20.2 (A), SW21.2
- new net: D15.2 (A), SW16.2
- new net: D10.2 (A), SW11.2
- new net: D5.2 (A), SW6.2
Other:
- moved on the sheet: U1

Commit message: some work
Parts:
- added J1: Conn_01x04_Male, symbol Conn_01x04_Male
Connections:
- net +3V3: now also J1.1 (Pin_1)
- net GND: now also J1.4 (Pin_4)
- net at U1.31 (SWDIO): now also J1.2 (Pin_2)
- net at U1.32 (SWCLK): now also J1.3 (Pin_3)
Changed lines of the file:
@@
 $EndComp
 $Comp
-L +3.3V #PWR01
+L +3.3V #PWR5
 U 1 1 59BBF369
 P 34400 -7050
-F 0 "#PWR01" H 34400 -7200 50  0001 C CNN
+F 0 "#PWR5" H 34400 -7200 50  0001 C CNN
 F 1 "+3.3V" H 34400 -6910 50  0000 C CNN
 F 2 "" H 34400 -7050 50  0001 C CNN
@@
 $EndComp
 $Comp
-L GND #PWR02
+L GND #PWR3
 U 1 1 59BBF383
 P 3150 7100
-F 0 "#PWR02" H 3150 6850 50  0001 C CNN
+F 0 "#PWR3" H 3150 6850 50  0001 C CNN
 F 1 "GND" H 3150 6950 50  0000 C CNN
 F 2 "" H 3150 7100 50  0001 C CNN
@@
 $EndComp
 $Comp
-L +3.3V #PWR03
+L +3.3V #PWR4
 U 1 1 59C15857
 P 5000 5950
-F 0 "#PWR03" H 5000 5800 50  0001 C CNN
+F 0 "#PWR4" H 5000 5800 50  0001 C CNN
 F 1 "+3.3V" H 5000 6090 50  0000 C CNN
 F 2 "" H 5000 5950 50  0001 C CNN
@@
 Connection ~ 2700 6350
 $Comp
-L +3.3V #PWR04
+L +3.3V #PWR2
 U 1 1 59C23ED5
 P 1600 650
-F 0 "#PWR04" H 1600 500 50  0001 C CNN
+F 0 "#PWR2" H 1600 500 50  0001 C CNN
 F 1 "+3.3V" H 1600 790 50  0000 C CNN
 F 2 "" H 1600 650 50  0001 C CNN
@@
 $EndComp
 $Comp
-L GND #PWR05
+L GND #PWR1
 U 1 1 59C23F89
 P 1350 2200
-F 0 "#PWR05" H 1350 1950 50  0001 C CNN
+F 0 "#PWR1" H 1350 1950 50  0001 C CNN
 F 1 "GND" H 1350 2050 50  0000 C CNN
 F 2 "" H 1350 2200 50  0001 C CNN
@@
 	2100 1900 1600 1900
 Wire Wire Line
-	1600 1900 1600 650
+	1600 650  1600 3450
+$Comp
+L Conn_01x04_Male J1
+U 1 1 59C3A25B
+P 1000 3550
+F 0 "J1" H 1000 3750 50  0000 C CNN
+F 1 "Conn_01x04_Male" H 1000 3250 50  0000 C CNN
+F 2 "" H 1000 3550 50  0001 C CNN
+F 3 "" H 1000 3550 50  0001 C CNN
+	1    1000 3550
+	1    0    0    -1
+$EndComp
+Wire Wire Line
+	1600 3450 1200 3450
+Connection ~ 1600 1900
+Wire Wire Line
+	1200 3550 4100 3550
+Wire Wire Line
+	4100 3550 4100 1300
+Wire Wire Line
+	4100 1300 4000 1300
+Wire Wire Line
+	1200 3650 4200 3650
+Wire Wire Line
+	4200 3650 4200 1200
+Wire Wire Line
+	4200 1200 4000 1200
+Wire Wire Line
+	1200 3750 1700 3750
+Wire Wire Line
+	1700 3750 1700 1800
+Connection ~ 1700 1800
 $EndSCHEMATC

Commit message: routing
Parts:
- removed D35, D9: D, Diodes_SMD:D_MiniMELF, symbol D
- removed SW1, SW10, SW36: MOM-SPST, Misc:CHERRY-MX, symbol MOM-SPST
- added D36: LED, LEDs:LED_1206, symbol LED
- added R4: R, Resistors_SMD:R_0805, symbol R
- BT1: footprint (none) -> Misc:KEYSTONE-82_AAA_battery-clip
- J1: footprint (none) -> Pin_Headers:Pin_Header_Angled_1x04_Pitch2.54mm
- L1: footprint (none) -> SMD_Packages:SMD-1206_Pol
- R1, R2, R3: footprint (none) -> Resistors_SMD:R_0805
- U1: footprint (none) -> Misc:Core51822(B)
Connections:
- wire segments 127 -> 151
Changed lines of the file:
@@
 LIBS:contrib
 LIBS:valves
-LIBS:nrf51822
-LIBS:mcp1640
-LIBS:switches
+LIBS:core51822b
 LIBS:interphase-cache
 EELAYER 25 0
@@
 F 0 "U1" H 3050 1400 60  0000 C CNN
 F 1 "Core51822B" H 3050 1250 60  0000 C CNN
-F 2 "" H 3050 1400 60  0001 C CNN
+F 2 "Misc:Core51822(B)" H 3050 1400 60  0001 C CNN
 F 3 "" H 3050 1400 60  0001 C CNN
 	1    3050 1300
@@
 F 0 "BT1" H 2450 6750 50  0000 L CNN
 F 1 "Battery_Cell" H 2450 6650 50  0000 L CNN
-F 2 "" V 2350 6710 50  0001 C CNN
+F 2 "Misc:KEYSTONE-82_AAA_battery-clip" V 2350 6710 50  0001 C CNN
 F 3 "" V 2350 6710 50  0001 C CNN
 	1    2350 6650
@@
 $EndComp
 $Comp
-L +3.3V #PWR5
+L +3.3V #PWR01
 U 1 1 59BBF369
 P 34400 -7050
-F 0 "#PWR5" H 34400 -7200 50  0001 C CNN
+F 0 "#PWR01" H 34400 -7200 50  0001 C CNN
 F 1 "+3.3V" H 34400 -6910 50  0000 C CNN
 F 2 "" H 34400 -7050 50  0001 C CNN
@@
 $EndComp
 $Comp
-L GND #PWR3
+L GND #PWR02
 U 1 1 59BBF383
 P 3150 7100
-F 0 "#PWR3" H 3150 6850 50  0001 C CNN
+F 0 "#PWR02" H 3150 6850 50  0001 C CNN
 F 1 "GND" H 3150 6950 50  0000 C CNN
 F 2 "" H 3150 7100 50  0001 C CNN
@@
 F 0 "L1" V 3400 5950 50  0000 C CNN
 F 1 "4,7µH" V 3525 5950 50  0000 C CNN
-F 2 "" H 3450 5950 50  0001 C CNN
+F 2 "SMD_Packages:SMD-1206_Pol" H 3450 5950 50  0001 C CNN
 F 3 "" H 3450 5950 50  0001 C CNN
 	1    3450 5950
@@
 F 0 "R1" V 4680 6300 50  0000 C CNN
 F 1 "536K" V 4600 6300 50  0000 C CNN
-F 2 "" V 4530 6300 50  0001 C CNN
+F 2 "Resistors_SMD:R_0805" V 4530 6300 50  0001 C CNN
 F 3 "" H 4600 6300 50  0001 C CNN
 	1    4600 6300
@@
 F 0 "R2" V 4680 6700 50  0000 C CNN
 F 1 "309K" V 4600 6700 50  0000 C CNN
-F 2 "" V 4530 6700 50  0001 C CNN
+F 2 "Resistors_SMD:R_0805" V 4530 6700 50  0001 C CNN
 F 3 "" H 4600 6700 50  0001 C CNN
 	1    4600 6700
@@
 F 3 "" H 5000 6500 50  0001 C CNN
 	1    5000 6500
-	1    0    0    -1
-$EndComp
-$Comp
-L MOM-SPST SW1
-U 1 1 59BFAFF8
-P 3400 6500
-F 0 "SW1" H 3475 6600 60  0000 L BNB
-F 1 "MOM-SPST" H 3475 6400 40  0000 L TNN
-F 2 "Misc:CHERRY-MX" H 3475 6325 40  0001 L TNN
-F 3 "" H 3300 6600 60  0001 C CNN
-F 4 "-" H 3475 6700 40  0001 L BNN "Part"
-F 5 "Switch" H 3475 6800 40  0001 L BNN "Family"
-	1    3400 6500
 	1    0    0    -1
 $EndComp
@@
 $EndComp
 $Comp
-L MOM-SPST SW10
-U 1 1 59BFC112
-P 7400 2900
-F 0 "SW10" H 7475 3000 60  0000 L BNB
-F 1 "MOM-SPST" H 7475 2800 40  0000 L TNN
-F 2 "Misc:CHERRY-MX" H 7475 2725 40  0001 L TNN
-F 3 "" H 7300 3000 60  0001 C CNN
-F 4 "-" H 7475 3100 40  0001 L BNN "Part"
-F 5 "Switch" H 7475 3200 40  0001 L BNN "Family"
-	1    7400 2900
-	1    0    0    -1
-$EndComp
-$Comp
 L MOM-SPST SW5
 U 1 1 59BFC11A
@@
 $EndComp
 $Comp
-L MOM-SPST SW36
-U 1 1 59BFC34C
-P 10400 3500
-F 0 "SW36" H 10475 3600 60  0000 L BNB
-F 1 "MOM-SPST" H 10475 3400 40  0000 L TNN
-F 2 "Misc:CHERRY-MX" H 10475 3325 40  0001 L TNN
-F 3 "" H 10300 3600 60  0001 C CNN
-F 4 "-" H 10475 3700 40  0001 L BNN "Part"
-F 5 "Switch" H 10475 3800 40  0001 L BNN "Family"
-	1    10400 3500
-	1    0    0    -1
-$EndComp
-$Comp
 L MOM-SPST SW31
 U 1 1 59BFC354
@@
 $EndComp
 $Comp
-L D D9
-U 1 1 59C10E1F
-P 7650 2900
-F 0 "D9" H 7650 3000 50  0000 C CNN
-F 1 "D" H 7650 2800 50  0000 C CNN
-F 2 "Diodes_SMD:D_MiniMELF" H 7650 2900 50  0001 C CNN
-F 3 "" H 7650 2900 50  0001 C CNN
-	1    7650 2900
-	-1   0    0    -1
-$EndComp
-$Comp
 L D D10
 U 1 1 59C10EF1
@@
 $EndComp
 $Comp
-L D D35
-U 1 1 59C11BF6
-P 10650 3500
-F 0 "D35" H 10650 3600 50  0000 C CNN
-F 1 "D" H 10650 3400 50  0000 C CNN
-F 2 "Diodes_SMD:D_MiniMELF" H 10650 3500 50  0001 C CNN
-F 3 "" H 10650 3500 50  0001 C CNN
-	1    10650 3500
-	-1   0    0    -1
-$EndComp
-$Comp
 L D D34
 U 1 1 59C11CF1
@@
 F 0 "R3" V 3630 6750 50  0000 C CNN
 F 1 "100K" V 3550 6750 50  0000 C CNN
-F 2 "" V 3480 6750 50  0001 C CNN
+F 2 "Resistors_SMD:R_0805" V 3480 6750 50  0001 C CNN
 F 3 "" H 3550 6750 50  0001 C CNN
 	1    3550 6750
@@
 $EndComp
 $Comp
-L +3.3V #PWR4
+L +3.3V #PWR03
 U 1 1 59C15857
 P 5000 5950
-F 0 "#PWR4" H 5000 5800 50  0001 C CNN
+F 0 "#PWR03" H 5000 5800 50  0001 C CNN
 F 1 "+3.3V" H 5000 6090 50  0000 C CNN
 F 2 "" H 5000 5950 50  0001 C CNN
@@
 Connection ~ 4600 6950
 Wire Wire Line
-	3500 6500 3550 6500
+	3300 6500 3550 6500
 Wire Wire Line
 	3300 6500 3300 6350
@@
 	6100 2600 10300 2600
 Wire Wire Line
-	10300 3200 10300 3500
-Wire Wire Line
-	6000 3200 10300 3200
-Wire Wire Line
 	6700 2300 6700 2000
 Connection ~ 6700 2000
@@
 Connection ~ 6700 3200
 Wire Wire Line
-	7300 3500 7300 3200
+	7300 3200 7300 3500
 Connection ~ 7300 3200
-Wire Wire Line
-	7300 2900 7300 2600
 Connection ~ 7300 2600
 Wire Wire Line
@@
 Connection ~ 7900 2600
 Wire Wire Line
-	7900 3500 7900 3200
+	7900 3200 7900 3500
 Connection ~ 7900 3200
 Wire Wire Line
-	8500 3500 8500 3200
+	8500 3200 8500 3500
 Connection ~ 8500 3200
 Wire Wire Line
@@
 Connection ~ 8500 2000
 Wire Wire Line
-	9100 3500 9100 3200
+	9100 3200 9100 3500
 Connection ~ 9100 3200
 Wire Wire Line
@@
 Connection ~ 9700 2600
 Wire Wire Line
-	9700 3500 9700 3200
+	9700 3200 9700 3500
 Connection ~ 9700 3200
 Wire Wire Line
@@
 Connection ~ 2700 6350
 $Comp
-L +3.3V #PWR2
+L +3.3V #PWR04
 U 1 1 59C23ED5
 P 1600 650
-F 0 "#PWR2" H 1600 500 50  0001 C CNN
+F 0 "#PWR04" H 1600 500 50  0001 C CNN
 F 1 "+3.3V" H 1600 790 50  0000 C CNN
 F 2 "" H 1600 650 50  0001 C CNN
@@
 $EndComp
 $Comp
-L GND #PWR1
+L GND #PWR05
 U 1 1 59C23F89
 P 1350 2200
-F 0 "#PWR1" H 1350 1950 50  0001 C CNN
+F 0 "#PWR05" H 1350 1950 50  0001 C CNN
 F 1 "GND" H 1350 2050 50  0000 C CNN
 F 2 "" H 1350 2200 50  0001 C CNN
@@
 $EndComp
 Wire Wire Line
-	2100 1800 1350 1800
+	1350 1800 2100 1800
 Wire Wire Line
 	1350 800  1350 2200
@@
 F 0 "J1" H 1000 3750 50  0000 C CNN
 F 1 "Conn_01x04_Male" H 1000 3250 50  0000 C CNN
-F 2 "" H 1000 3550 50  0001 C CNN
+F 2 "Pin_Headers:Pin_Header_Angled_1x04_Pitch2.54mm" H 1000 3550 50  0001 C CNN
 F 3 "" H 1000 3550 50  0001 C CNN
 	1    1000 3550
@@
 	1700 3750 1700 1800
 Connection ~ 1700 1800
+$Comp
+L LED D36
+U 1 1 59C53D55
+P 3000 2700
+F 0 "D36" H 3000 2800 50  0000 C CNN
+F 1 "LED" H 3000 2600 50  0000 C CNN
+F 2 "LEDs:LED_1206" H 3000 2700 50  0001 C CNN
+F 3 "" H 3000 2700 50  0001 C CNN
+	1    3000 2700
+	0    -1   -1   0
+$EndComp
+$Comp
+L R R4
+U 1 1 59C53EAE
+P 3000 3100
+F 0 "R4" V 3080 3100 50  0000 C CNN
+F 1 "R" V 3000 3100 50  0000 C CNN
+F 2 "Resistors_SMD:R_0805" V 2930 3100 50  0001 C CNN
+F 3 "" H 3000 3100 50  0001 C CNN
+	1    3000 3100
+	1    0    0    -1
+$EndComp
+Wire Wire Line
+	3000 2550 3000 2500
+Wire Wire Line
+	3000 2500 2800 2500
+Wire Wire Line
+	2800 2500 2800 2350
+Wire Wire Line
+	3000 2850 3000 2950
+$Comp
+L GND #PWR06
+U 1 1 59C54565
+P 3000 3800
+F 0 "#PWR06" H 3000 3550 50  0001 C CNN
+F 1 "GND" H 3000 3650 50  0000 C CNN
+F 2 "" H 3000 3800 50  0001 C CNN
+F 3 "" H 3000 3800 50  0001 C CNN
+	1    3000 3800
+	1    0    0    -1
+$EndComp
+Wire Wire Line
+	3000 3250 3000 3800
+Wire Wire Line
+	6000 3200 9700 3200
+Wire Wire Line
+	7800 1700 7850 1700
+Connection ~ 7850 1700
+Wire Wire Line
+	7800 2300 7850 2300
+Connection ~ 7850 2300
+Wire Wire Line
+	7800 3500 7850 3500
+Connection ~ 7850 3500
+Wire Wire Line
+	8400 3500 8450 3500
+Connection ~ 8450 3500
+Wire Wire Line
+	8400 2900 8450 2900
+Connection ~ 8450 2900
+Wire Wire Line
+	8400 2300 8450 2300
+Connection ~ 8450 2300
+Wire Wire Line
+	8400 1700 8450 1700
+Connection ~ 8450 1700
+Wire Wire Line
+	9000 2300 9050 2300
+Connection ~ 9050 2300
+Wire Wire Line
+	9000 2900 9050 2900
+Connection ~ 9050 2900
+Wire Wire Line
+	9000 3500 9050 3500
+Connection ~ 9050 3500
+Wire Wire Line
+	9600 3500 9650 3500
+Connection ~ 9650 3500
+Wire Wire Line
+	9600 2900 9650 2900
+Connection ~ 9650 2900
+Wire Wire Line
+	9600 2300 9650 2300
+Connection ~ 9650 2300
+Wire Wire Line
+	9600 1700 9650 1700
+Connection ~ 9650 1700
+Wire Wire Line
+	10200 1700 10250 1700
+Connection ~ 10250 1700
+Wire Wire Line
+	10200 2300 10250 2300
+Connection ~ 10250 2300
+Wire Wire Line
+	10200 2900 10250 2900
+Connection ~ 10250 2900
+Wire Wire Line
+	10200 3500 10250 3500
+Connection ~ 10250 3500
+Wire Wire Line
+	10800 1700 10850 1700
+Connection ~ 10850 1700
+Wire Wire Line
+	10800 2300 10850 2300
+Connection ~ 10850 2300
+Wire Wire Line
+	10800 2900 10850 2900
+Connection ~ 10850 2900
 $EndSCHEMATC
