File: interphase.sch (KiCad schematic (older format))
At the start: 78 parts, among them J1 Conn_01x04_Male, SW11 MOM-SPST, SW12 MOM-SPST, SW13 MOM-SPST, SW14 MOM-SPST, SW15 MOM-SPST, SW16 MOM-SPST, SW17 MOM-SPST, SW18 MOM-SPST, SW19 MOM-SPST, SW2 MOM-SPST, SW20 MOM-SPST, SW21 MOM-SPST, SW22 MOM-SPST, SW23 MOM-SPST, SW24 MOM-SPST, SW25 MOM-SPST, SW26 MOM-SPST, SW27 MOM-SPST, SW28 MOM-SPST, SW29 MOM-SPST, SW3 MOM-SPST, SW30 MOM-SPST, SW31 MOM-SPST, SW32 MOM-SPST, SW33 MOM-SPST, SW34 MOM-SPST, SW35 MOM-SPST, SW4 MOM-SPST, SW5 MOM-SPST, SW6 MOM-SPST, SW7 MOM-SPST, SW8 MOM-SPST, SW9 MOM-SPST, U1 Core51822B, U2 MCP1640

Commit message: wololo
Parts:
- SW11, SW12, SW13, SW14, SW15, SW16, SW17, SW18, SW19, SW2, SW20, SW21, SW22, SW23, SW24, SW25, SW26, SW27, SW28, SW29, SW3, SW30, SW31, SW32, SW33, SW34, SW35, SW4, SW6, SW7, SW8, SW9: footprint Misc:CHERRY-MX -> Misc:CHERRY-MX_double_bo
- SW5: footprint Misc:CHERRY-MX -> Misc:CHERRY-MX_double_bo_2u
Connections:
- wire segments 151 -> 152
Changed lines of the file:
@@
 F 0 "SW32" H 10475 1200 60  0000 L BNB
 F 1 "MOM-SPST" H 10475 1000 40  0000 L TNN
-F 2 "Misc:CHERRY-MX" H 10475 925 40  0001 L TNN
+F 2 "Misc:CHERRY-MX_double_bo" H 10475 925 40  0001 L TNN
 F 3 "" H 10300 1200 60  0001 C CNN
 F 4 "-" H 10475 1300 40  0001 L BNN "Part"
@@
 F 0 "SW27" H 9875 1200 60  0000 L BNB
 F 1 "MOM-SPST" H 9875 1000 40  0000 L TNN
-F 2 "Misc:CHERRY-MX" H 9875 925 40  0001 L TNN
+F 2 "Misc:CHERRY-MX_double_bo" H 9875 925 40  0001 L TNN
 F 3 "" H 9700 1200 60  0001 C CNN
 F 4 "-" H 9875 1300 40  0001 L BNN "Part"
@@
 F 0 "SW22" H 9275 1200 60  0000 L BNB
 F 1 "MOM-SPST" H 9275 1000 40  0000 L TNN
-F 2 "Misc:CHERRY-MX" H 9275 925 40  0001 L TNN
+F 2 "Misc:CHERRY-MX_double_bo" H 9275 925 40  0001 L TNN
 F 3 "" H 9100 1200 60  0001 C CNN
 F 4 "-" H 9275 1300 40  0001 L BNN "Part"
@@
 F 0 "SW17" H 8675 1200 60  0000 L BNB
 F 1 "MOM-SPST" H 8675 1000 40  0000 L TNN
-F 2 "Misc:CHERRY-MX" H 8675 925 40  0001 L TNN
+F 2 "Misc:CHERRY-MX_double_bo" H 8675 925 40  0001 L TNN
 F 3 "" H 8500 1200 60  0001 C CNN
 F 4 "-" H 8675 1300 40  0001 L BNN "Part"
@@
 F 0 "SW12" H 8075 1200 60  0000 L BNB
 F 1 "MOM-SPST" H 8075 1000 40  0000 L TNN
-F 2 "Misc:CHERRY-MX" H 8075 925 40  0001 L TNN
+F 2 "Misc:CHERRY-MX_double_bo" H 8075 925 40  0001 L TNN
 F 3 "" H 7900 1200 60  0001 C CNN
 F 4 "-" H 8075 1300 40  0001 L BNN "Part"
@@
 F 0 "SW7" H 7475 1200 60  0000 L BNB
 F 1 "MOM-SPST" H 7475 1000 40  0000 L TNN
-F 2 "Misc:CHERRY-MX" H 7475 925 40  0001 L TNN
+F 2 "Misc:CHERRY-MX_double_bo" H 7475 925 40  0001 L TNN
 F 3 "" H 7300 1200 60  0001 C CNN
 F 4 "-" H 7475 1300 40  0001 L BNN "Part"
@@
 F 0 "SW2" H 6875 1200 60  0000 L BNB
 F 1 "MOM-SPST" H 6875 1000 40  0000 L TNN
-F 2 "Misc:CHERRY-MX" H 6875 925 40  0001 L TNN
+F 2 "Misc:CHERRY-MX_double_bo" H 6875 925 40  0001 L TNN
 F 3 "" H 6700 1200 60  0001 C CNN
 F 4 "-" H 6875 1300 40  0001 L BNN "Part"
@@
 F 0 "SW33" H 10475 1800 60  0000 L BNB
 F 1 "MOM-SPST" H 10475 1600 40  0000 L TNN
-F 2 "Misc:CHERRY-MX" H 10475 1525 40  0001 L TNN
+F 2 "Misc:CHERRY-MX_double_bo" H 10475 1525 40  0001 L TNN
 F 3 "" H 10300 1800 60  0001 C CNN
 F 4 "-" H 10475 1900 40  0001 L BNN "Part"
@@
 F 0 "SW28" H 9875 1800 60  0000 L BNB
 F 1 "MOM-SPST" H 9875 1600 40  0000 L TNN
-F 2 "Misc:CHERRY-MX" H 9875 1525 40  0001 L TNN
+F 2 "Misc:CHERRY-MX_double_bo" H 9875 1525 40  0001 L TNN
 F 3 "" H 9700 1800 60  0001 C CNN
 F 4 "-" H 9875 1900 40  0001 L BNN "Part"
@@
 F 0 "SW23" H 9275 1800 60  0000 L BNB
 F 1 "MOM-SPST" H 9275 1600 40  0000 L TNN
-F 2 "Misc:CHERRY-MX" H 9275 1525 40  0001 L TNN
+F 2 "Misc:CHERRY-MX_double_bo" H 9275 1525 40  0001 L TNN
 F 3 "" H 9100 1800 60  0001 C CNN
 F 4 "-" H 9275 1900 40  0001 L BNN "Part"
@@
 F 0 "SW18" H 8675 1800 60  0000 L BNB
 F 1 "MOM-SPST" H 8675 1600 40  0000 L TNN
-F 2 "Misc:CHERRY-MX" H 8675 1525 40  0001 L TNN
+F 2 "Misc:CHERRY-MX_double_bo" H 8675 1525 40  0001 L TNN
 F 3 "" H 8500 1800 60  0001 C CNN
 F 4 "-" H 8675 1900 40  0001 L BNN "Part"
@@
 F 0 "SW13" H 8075 1800 60  0000 L BNB
 F 1 "MOM-SPST" H 8075 1600 40  0000 L TNN
-F 2 "Misc:CHERRY-MX" H 8075 1525 40  0001 L TNN
+F 2 "Misc:CHERRY-MX_double_bo" H 8075 1525 40  0001 L TNN
 F 3 "" H 7900 1800 60  0001 C CNN
 F 4 "-" H 8075 1900 40  0001 L BNN "Part"
@@
 F 0 "SW8" H 7475 1800 60  0000 L BNB
 F 1 "MOM-SPST" H 7475 1600 40  0000 L TNN
-F 2 "Misc:CHERRY-MX" H 7475 1525 40  0001 L TNN
+F 2 "Misc:CHERRY-MX_double_bo" H 7475 1525 40  0001 L TNN
 F 3 "" H 7300 1800 60  0001 C CNN
 F 4 "-" H 7475 1900 40  0001 L BNN "Part"
@@
 F 0 "SW3" H 6875 1800 60  0000 L BNB
 F 1 "MOM-SPST" H 6875 1600 40  0000 L TNN
-F 2 "Misc:CHERRY-MX" H 6875 1525 40  0001 L TNN
+F 2 "Misc:CHERRY-MX_double_bo" H 6875 1525 40  0001 L TNN
 F 3 "" H 6700 1800 60  0001 C CNN
 F 4 "-" H 6875 1900 40  0001 L BNN "Part"
@@
 F 0 "SW34" H 10475 2400 60  0000 L BNB
 F 1 "MOM-SPST" H 10475 2200 40  0000 L TNN
-F 2 "Misc:CHERRY-MX" H 10475 2125 40  0001 L TNN
+F 2 "Misc:CHERRY-MX_double_bo" H 10475 2125 40  0001 L TNN
 F 3 "" H 10300 2400 60  0001 C CNN
 F 4 "-" H 10475 2500 40  0001 L BNN "Part"
@@
 F 0 "SW29" H 9875 2400 60  0000 L BNB
 F 1 "MOM-SPST" H 9875 2200 40  0000 L TNN
-F 2 "Misc:CHERRY-MX" H 9875 2125 40  0001 L TNN
+F 2 "Misc:CHERRY-MX_double_bo" H 9875 2125 40  0001 L TNN
 F 3 "" H 9700 2400 60  0001 C CNN
 F 4 "-" H 9875 2500 40  0001 L BNN "Part"
@@
 F 0 "SW24" H 9275 2400 60  0000 L BNB
 F 1 "MOM-SPST" H 9275 2200 40  0000 L TNN
-F 2 "Misc:CHERRY-MX" H 9275 2125 40  0001 L TNN
+F 2 "Misc:CHERRY-MX_double_bo" H 9275 2125 40  0001 L TNN
 F 3 "" H 9100 2400 60  0001 C CNN
 F 4 "-" H 9275 2500 40  0001 L BNN "Part"
@@
 F 0 "SW19" H 8675 2400 60  0000 L BNB
 F 1 "MOM-SPST" H 8675 2200 40  0000 L TNN
-F 2 "Misc:CHERRY-MX" H 8675 2125 40  0001 L TNN
+F 2 "Misc:CHERRY-MX_double_bo" H 8675 2125 40  0001 L TNN
 F 3 "" H 8500 2400 60  0001 C CNN
 F 4 "-" H 8675 2500 40  0001 L BNN "Part"
@@
 F 0 "SW14" H 8075 2400 60  0000 L BNB
 F 1 "MOM-SPST" H 8075 2200 40  0000 L TNN
-F 2 "Misc:CHERRY-MX" H 8075 2125 40  0001 L TNN
+F 2 "Misc:CHERRY-MX_double_bo" H 8075 2125 40  0001 L TNN
 F 3 "" H 7900 2400 60  0001 C CNN
 F 4 "-" H 8075 2500 40  0001 L BNN "Part"
@@
 F 0 "SW9" H 7475 2400 60  0000 L BNB
 F 1 "MOM-SPST" H 7475 2200 40  0000 L TNN
-F 2 "Misc:CHERRY-MX" H 7475 2125 40  0001 L TNN
+F 2 "Misc:CHERRY-MX_double_bo" H 7475 2125 40  0001 L TNN
 F 3 "" H 7300 2400 60  0001 C CNN
 F 4 "-" H 7475 2500 40  0001 L BNN "Part"
@@
 F 0 "SW4" H 6875 2400 60  0000 L BNB
 F 1 "MOM-SPST" H 6875 2200 40  0000 L TNN
-F 2 "Misc:CHERRY-MX" H 6875 2125 40  0001 L TNN
+F 2 "Misc:CHERRY-MX_double_bo" H 6875 2125 40  0001 L TNN
 F 3 "" H 6700 2400 60  0001 C CNN
 F 4 "-" H 6875 2500 40  0001 L BNN "Part"
@@
 F 0 "SW35" H 10475 3000 60  0000 L BNB
 F 1 "MOM-SPST" H 10475 2800 40  0000 L TNN
-F 2 "Misc:CHERRY-MX" H 10475 2725 40  0001 L TNN
+F 2 "Misc:CHERRY-MX_double_bo" H 10475 2725 40  0001 L TNN
 F 3 "" H 10300 3000 60  0001 C CNN
 F 4 "-" H 10475 3100 40  0001 L BNN "Part"
@@
 F 0 "SW30" H 9875 3000 60  0000 L BNB
 F 1 "MOM-SPST" H 9875 2800 40  0000 L TNN
-F 2 "Misc:CHERRY-MX" H 9875 2725 40  0001 L TNN
+F 2 "Misc:CHERRY-MX_double_bo" H 9875 2725 40  0001 L TNN
 F 3 "" H 9700 3000 60  0001 C CNN
 F 4 "-" H 9875 3100 40  0001 L BNN "Part"
@@
 F 0 "SW25" H 9275 3000 60  0000 L BNB
 F 1 "MOM-SPST" H 9275 2800 40  0000 L TNN
-F 2 "Misc:CHERRY-MX" H 9275 2725 40  0001 L TNN
+F 2 "Misc:CHERRY-MX_double_bo" H 9275 2725 40  0001 L TNN
 F 3 "" H 9100 3000 60  0001 C CNN
 F 4 "-" H 9275 3100 40  0001 L BNN "Part"
@@
 F 0 "SW20" H 8675 3000 60  0000 L BNB
 F 1 "MOM-SPST" H 8675 2800 40  0000 L TNN
-F 2 "Misc:CHERRY-MX" H 8675 2725 40  0001 L TNN
+F 2 "Misc:CHERRY-MX_double_bo" H 8675 2725 40  0001 L TNN
 F 3 "" H 8500 3000 60  0001 C CNN
 F 4 "-" H 8675 3100 40  0001 L BNN "Part"
@@
 F 0 "SW15" H 8075 3000 60  0000 L BNB
 F 1 "MOM-SPST" H 8075 2800 40  0000 L TNN
-F 2 "Misc:CHERRY-MX" H 8075 2725 40  0001 L TNN
+F 2 "Misc:CHERRY-MX_double_bo" H 8075 2725 40  0001 L TNN
 F 3 "" H 7900 3000 60  0001 C CNN
 F 4 "-" H 8075 3100 40  0001 L BNN "Part"
@@
 F 0 "SW5" H 6875 3000 60  0000 L BNB
 F 1 "MOM-SPST" H 6875 2800 40  0000 L TNN
-F 2 "Misc:CHERRY-MX" H 6875 2725 40  0001 L TNN
+F 2 "Misc:CHERRY-MX_double_bo_2u" H 6875 2725 40  0001 L TNN
 F 3 "" H 6700 3000 60  0001 C CNN
 F 4 "-" H 6875 3100 40  0001 L BNN "Part"
@@
 F 0 "SW31" H 9875 3600 60  0000 L BNB
 F 1 "MOM-SPST" H 9875 3400 40  0000 L TNN
-F 2 "Misc:CHERRY-MX" H 9875 3325 40  0001 L TNN
+F 2 "Misc:CHERRY-MX_double_bo" H 9875 3325 40  0001 L TNN
 F 3 "" H 9700 3600 60  0001 C CNN
 F 4 "-" H 9875 3700 40  0001 L BNN "Part"
@@
 F 0 "SW26" H 9275 3600 60  0000 L BNB
 F 1 "MOM-SPST" H 9275 3400 40  0000 L TNN
-F 2 "Misc:CHERRY-MX" H 9275 3325 40  0001 L TNN
+F 2 "Misc:CHERRY-MX_double_bo" H 9275 3325 40  0001 L TNN
 F 3 "" H 9100 3600 60  0001 C CNN
 F 4 "-" H 9275 3700 40  0001 L BNN "Part"
@@
 F 0 "SW21" H 8675 3600 60  0000 L BNB
 F 1 "MOM-SPST" H 8675 3400 40  0000 L TNN
-F 2 "Misc:CHERRY-MX" H 8675 3325 40  0001 L TNN
+F 2 "Misc:CHERRY-MX_double_bo" H 8675 3325 40  0001 L TNN
 F 3 "" H 8500 3600 60  0001 C CNN
 F 4 "-" H 8675 3700 40  0001 L BNN "Part"
@@
 F 0 "SW16" H 8075 3600 60  0000 L BNB
 F 1 "MOM-SPST" H 8075 3400 40  0000 L TNN
-F 2 "Misc:CHERRY-MX" H 8075 3325 40  0001 L TNN
+F 2 "Misc:CHERRY-MX_double_bo" H 8075 3325 40  0001 L TNN
 F 3 "" H 7900 3600 60  0001 C CNN
 F 4 "-" H 8075 3700 40  0001 L BNN "Part"
@@
 F 0 "SW11" H 7475 3600 60  0000 L BNB
 F 1 "MOM-SPST" H 7475 3400 40  0000 L TNN
-F 2 "Misc:CHERRY-MX" H 7475 3325 40  0001 L TNN
+F 2 "Misc:CHERRY-MX_double_bo" H 7475 3325 40  0001 L TNN
 F 3 "" H 7300 3600 60  0001 C CNN
 F 4 "-" H 7475 3700 40  0001 L BNN "Part"
@@
 F 0 "SW6" H 6875 3600 60  0000 L BNB
 F 1 "MOM-SPST" H 6875 3400 40  0000 L TNN
-F 2 "Misc:CHERRY-MX" H 6875 3325 40  0001 L TNN
+F 2 "Misc:CHERRY-MX_double_bo" H 6875 3325 40  0001 L TNN
 F 3 "" H 6700 3600 60  0001 C CNN
 F 4 "-" H 6875 3700 40  0001 L BNN "Part"
@@
 	10800 2900 10850 2900
 Connection ~ 10850 2900
+Wire Wire Line
+	9000 1700 9050 1700
+Connection ~ 9050 1700
 $EndSCHEMATC

Commit message: finish layout and fix prototype issues
Parts:
- removed D36: LED, LEDs:LED_1206, symbol LED
- removed R3: 100K, Resistors_SMD:R_0805, symbol R
- removed R4: R, Resistors_SMD:R_0805, symbol R
- added C3: 4,7µF, Capacitors_SMD:C_0805_HandSoldering, symbol C
- added C4: 10µF, Capacitors_SMD:C_0805_HandSoldering, symbol C
- added D35, D36, D37, D38, D39, D40, D41, D42, D43, D44, D45, D46, D47, D48, D49, D50, D51, D52, D53, D54, D55, D56, D57, D58, D59, D60, D61, D62, D63, D64, D65, D66, D9: D, Diodes_SMD:D_MiniMELF, symbol D
- added L2: 4,7µH, SMD_Packages:SMD-1206_Pol, symbol L
- added R6: 536K, Resistors_SMD:R_0805, symbol R
- added R7: 309K, Resistors_SMD:R_0805, symbol R
- added U3: MCP1640, TO_SOT_Packages_SMD:SOT-23-6, symbol MCP1640
- added U4: Core51822B, Misc:Core51822(B), symbol Core51822B
- SW11, SW12, SW13, SW14, SW15, SW16, SW17, SW18, SW19, SW2, SW20, SW21, SW22, SW23, SW24, SW25, SW27, SW28, SW29, SW3, SW30, SW32, SW33, SW34, SW35, SW4, SW6, SW7, SW8, SW9: footprint Misc:CHERRY-MX_double_bo -> Misc:CHERRY-MX_double_bo_nodiode
- SW26, SW31: footprint Misc:CHERRY-MX_double_bo -> Misc:CHERRY-MX_double_bo_1_5u
- SW5: footprint Misc:CHERRY-MX_double_bo_2u -> Misc:CHERRY-MX_double_bo_2u_nodiode
Connections:
- net labels added: +BATT
- wire segments 152 -> 287
Other:
- moved on the sheet: BT1, C1, C2, D1, D10, D11, D12, D13, D14, D15, D16, D17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
